Commit message: final version

File: urdf/myfirst.urdf (robot description, URDF)
Before this commit: robot myfirst, 1 links, 0 joints
Links:
- added link head; visual sphere radius=0.2
- added link left_eye; visual sphere radius=0.02
- added link right_eye; visual sphere radius=0.02
Joints:
- added joint head_to_base: type continuous, parent base_link, child head, origin xyz=0 0 0.3, axis 0 0 1
- added joint head_to_left_eye: type fixed, parent head, child left_eye, origin xyz=-0.05 0.2 0.05
- added joint head_to_right_eye: type fixed, parent head, child right_eye, origin xyz=0.05 0.2 0.05
